Commit message: Applied optical center frame to Z axis forward | fixed namespaces prefixes
Signed-off-by: Jakub Delicat <jakub.delicat@husarion.com>

File: urdf/stereolabs_zed.urdf.xacro (robot description, xacro)
@@ -111,5 +111,5 @@
       <parent link="${device_namespace}_center" />
       <child link="${device_namespace}_center_optical_frame" />
-      <origin xyz="0.01 0 0" rpy="0 0 0" />
+      <origin xyz="0.01 0 0" rpy="${-pi/2.0} 0 ${-pi/2.0}" />
     </joint>
     <!-- Left Camera -->
@@ -163,5 +163,5 @@
     camera
       should be more accurate different frames and fovs can be set -->
-    <gazebo reference="${device_namespace}_center_optical_frame">
+    <gazebo reference="${device_namespace}_link">
       <sensor type="camera" name="${ns}${device_namespace}_stereolabs_zed_color">
         <always_on>true</always_on>
@@ -169,5 +169,5 @@
         <topic>${ns}${device_namespace}/zed_node/rgb/image_rect_color</topic>
         <visualize>false</visualize>
-        <ignition_frame_id>${device_namespace}_center_optical_frame</ignition_frame_id>
+        <ignition_frame_id>${ns}${device_namespace}_center_optical_frame</ignition_frame_id>
         <camera>
           <horizontal_fov>${110.0/180.0*pi}</horizontal_fov>
@@ -188,5 +188,5 @@
         <topic>${ns}${device_namespace}/zed_node/depth</topic>
         <visualize>false</visualize>
-        <ignition_frame_id>${device_namespace}_center_optical_frame</ignition_frame_id>
+        <ignition_frame_id>${ns}${device_namespace}_center_optical_frame</ignition_frame_id>
         <camera>
           <horizontal_fov>${110.0/180.0*pi}</horizontal_fov>

Commit message: Fixed zed
Signed-off-by: Jakub Delicat <jakub.delicat@husarion.com>

File: urdf/stereolabs_zed.urdf.xacro (robot description, xacro)
@@ -87,5 +87,6 @@
     <link name="${device_namespace}_center">
       <visual>
-        <origin xyz="${screw_offset_x} 0 ${screw_offset_z}" rpy="0 0 0" />
+        <!-- 0.02 in x is caused because the visual model is in the frame -->
+        <origin xyz="${screw_offset_x-0.02} 0 ${screw_offset_z}" rpy="0 0 0" />
         <geometry>
           <mesh filename="package://ros_components_description/meshes/${model}.stl" />
@@ -104,5 +105,6 @@
       <parent link="${device_namespace}_link" />
       <child link="${device_namespace}_center" />
-      <origin xyz="0 0 ${height/2}" rpy="0 ${bottom_slope} 0" />
+      <!-- 0.02 in x is caused because the visual model is in the frame -->
+      <origin xyz="0.02 0 ${height/2}" rpy="0 ${bottom_slope} 0" />
     </joint>
     <!-- Artificially Created Camera Center -->
@@ -111,5 +113,5 @@
       <parent link="${device_namespace}_center" />
       <child link="${device_namespace}_center_optical_frame" />
-      <origin xyz="0.01 0 0" rpy="${-pi/2.0} 0 ${-pi/2.0}" />
+      <origin xyz="0.0 0.0 0.0" rpy="${-pi/2.0} 0 ${-pi/2.0}" />
     </joint>
     <!-- Left Camera -->
@@ -163,5 +165,5 @@
     camera
       should be more accurate different frames and fovs can be set -->
-    <gazebo reference="${device_namespace}_link">
+    <gazebo reference="${device_namespace}_center">
       <sensor type="camera" name="${ns}${device_namespace}_stereolabs_zed_color">
         <always_on>true</always_on>
